Commit message: Modified xacro and world files to get kinect, hokuyo, etc. working with MACE and ROS.

File: catkin_sim_environment/src/sim_vehicles_description/urdf/basic_quadrotor/basic_quadrotor_asus.urdf.xacro (robot description, xacro)
@@ -3,12 +3,7 @@
     <xacro:property name="M_PI" value="3.1415926535897931" />
     <!-- Included URDF Files -->
-    <xacro:include filename="$(find sim_vehicles_description)/urdf/basic_quadrotor/quadrotor_base.urdf.xacro" />
+    <xacro:include filename="$(find sim_vehicles_description)/urdf/basic_quadrotor/basic_quadrotor_base.urdf.xacro" />
     <!-- Instantiate quadrotor_base_macro once (has no parameters atm) -->
     <xacro:quadrotor_base_macro />
-    <!-- Hokuyo UTM-30LX mounted upside down below the quadrotor body -->
-    <xacro:include filename="$(find sim_sensors_description)/urdf/hokuyo_utm30lx.urdf.xacro" />
-    <xacro:hokuyo_utm30lx name="laser0" parent="base_link" ros_topic="scan" update_rate="40" ray_count="1081" min_angle="-135" max_angle="135">
-      <origin xyz="0.0 0.0 -0.097" rpy="${M_PI} 0 0"/>
-    </xacro:hokuyo_utm30lx>
     <!-- Asus Xiton Live Pro -->
     <xacro:include filename="$(find sim_sensors_description)/urdf/asus_camera.urdf.xacro" />

File: catkin_sim_environment/src/sim_vehicles_description/urdf/basic_quadrotor/basic_quadrotor_asus_with_hokuyo_utm30lx.urdf.xacro (robot description, xacro)
@@ -3,7 +3,12 @@
     <xacro:property name="M_PI" value="3.1415926535897931" />
     <!-- Included URDF Files -->
-    <xacro:include filename="$(find sim_vehicles_description)/urdf/basic_quadrotor/quadrotor_base.urdf.xacro" />
+    <xacro:include filename="$(find sim_vehicles_description)/urdf/basic_quadrotor/basic_quadrotor_base.urdf.xacro" />
     <!-- Instantiate quadrotor_base_macro once (has no parameters atm) -->
     <xacro:quadrotor_base_macro />
+    <!-- Hokuyo UTM-30LX mounted upside down below the quadrotor body -->
+    <xacro:include filename="$(find sim_sensors_description)/urdf/hokuyo_utm30lx.urdf.xacro" />
+    <xacro:hokuyo_utm30lx name="laser0" parent="base_link" ros_topic="scan" update_rate="40" ray_count="1081" min_angle="-135" max_angle="135">
+      <origin xyz="0.0 0.0 -0.097" rpy="${M_PI} 0 0"/>
+    </xacro:hokuyo_utm30lx>
     <!-- Asus Xiton Live Pro -->
     <xacro:include filename="$(find sim_sensors_description)/urdf/asus_camera.urdf.xacro" />

File: catkin_sim_environment/src/sim_vehicles_description/urdf/basic_quadrotor/basic_quadrotor_cam.urdf.xacro (robot description, xacro)
@@ -3,5 +3,5 @@
     <xacro:property name="M_PI" value="3.1415926535897931" />
     <!-- Included URDF Files -->
-    <xacro:include filename="$(find sim_vehicles_description)/urdf/basic_quadrotor/quadrotor_base.urdf.xacro" />
+    <xacro:include filename="$(find sim_vehicles_description)/urdf/basic_quadrotor/basic_quadrotor_base.urdf.xacro" />
     <!-- Instantiate quadrotor_base_macro once (has no parameters atm) -->
     <xacro:quadrotor_base_macro />

File: catkin_sim_environment/src/sim_vehicles_description/urdf/basic_quadrotor/basic_quadrotor_hokuyo_utm30lx.urdf.xacro (robot description, xacro)
@@ -3,5 +3,5 @@
     <xacro:property name="M_PI" value="3.1415926535897931" />
     <!-- Included URDF Files -->
-    <xacro:include filename="$(find sim_vehicles_description)/urdf/basic_quadrotor/quadrotor_base.urdf.xacro" />
+    <xacro:include filename="$(find sim_vehicles_description)/urdf/basic_quadrotor/basic_quadrotor_base.urdf.xacro" />
     <!-- Instantiate quadrotor_base_macro once (has no parameters atm) -->
     <xacro:quadrotor_base_macro />

File: catkin_sim_environment/src/sim_vehicles_description/urdf/basic_quadrotor/basic_quadrotor_kinect.urdf.xacro (robot description, xacro)
@@ -3,5 +3,5 @@
     <xacro:property name="M_PI" value="3.1415926535897931" />
     <!-- Included URDF Files -->
-    <xacro:include filename="$(find sim_vehicles_description)/urdf/basic_quadrotor/quadrotor_base.urdf.xacro" />
+    <xacro:include filename="$(find sim_vehicles_description)/urdf/basic_quadrotor/basic_quadrotor_base.urdf.xacro" />
     <!-- Instantiate quadrotor_base_macro once (has no parameters atm) -->
     <xacro:quadrotor_base_macro />
