Commit message: Moving hokuyo to top of the quadrotor to miss the legs when scanning

File: catkin_sim_environment/src/sim_vehicles_description/urdf/basic_quadrotor/basic_quadrotor_hokuyo_utm30lx.urdf.xacro (robot description, xacro)
@@ -9,5 +9,5 @@
     <xacro:include filename="$(find sim_sensors_description)/urdf/hokuyo_utm30lx.urdf.xacro" />
     <xacro:hokuyo_utm30lx name="laser0" parent="base_link" ros_topic="scan" update_rate="40" ray_count="1081" min_angle="-135" max_angle="135">
-      <origin xyz="0.0 0.0 -0.097" rpy="${M_PI} 0 0"/>
+      <origin xyz="0.0 0.0 0.070" rpy="${M_PI} 0 0"/>
     </xacro:hokuyo_utm30lx>
     <!-- Forward facing camera -->
