Commit message: multi_basic_quadrotor scripts work. TODO: 1) Move from bash to python for ease of use in the future. 2) Document launch process. 3) Make sure ROS module handles multiple vehicles properly

File: catkin_sim_environment/src/sim_sensors_description/urdf/generic_thermal_camera.urdf.xacro (robot description, xacro)
@@ -1,5 +1,5 @@
 <?xml version="1.0"?>
 <robot xmlns:xacro="http://ros.org/wiki/xacro">
-  <xacro:include filename="$(find hector_xacro_tools)/urdf/sensor_macros.urdf.xacro" />
+<!--  <xacro:include filename="$(find hector_xacro_tools)/urdf/sensor_macros.urdf.xacro" /> -->
   <xacro:macro name="generic_thermal_camera" params="name parent *origin">
     <joint name="${name}_joint" type="fixed">

File: catkin_sim_environment/src/sim_sensors_description/urdf/sonar_sensor.urdf.xacro (robot description, xacro)
@@ -17,5 +17,5 @@
         <geometry>
           <!--<box size="0.01 0.01 0.01" /> -->
-          <mesh filename="package://hector_sensors_description/meshes/sonar_sensor/max_sonar_ez4.dae"/>
+          <mesh filename="package://sim_sensors_description/meshes/sonar_sensor/max_sonar_ez4.dae"/>
         </geometry>
       </visual>
